Commit message: Add cone models and FLW cone track world

File: packages/src/roboracer_gazebo/models/f110_car/f110_car.urdf (robot description, URDF)
Before this commit: robot f110_car, 12 links, 11 joints
Links:
- link camera: geometry collision box size=0.03 0.17 0.03; visual mesh filename=file:///home/dhanush/rrstack/packages/src/roboracer_gazebo/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
- link chassis: geometry collision box size=0.49 0.18 0.1; visual mesh filename=file:///home/dhanush/rrstack/packages/src/roboracer_gazebo/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
- link laser: geometry collision box size=0.1 0.1 0.1; visual mesh filename=file:///home/dhanush/rrstack/packages/src/roboracer_gazebo/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
- link left_wheel_back: geometry collision cylinder length=0.045 radius=0.05; visual mesh filename=file:///home/dhanush/rrstack/packages/src/roboracer_gazebo/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
- link left_wheel_front: geometry collision cylinder length=0.045 radius=0.05; visual mesh filename=file:///home/dhanush/rrstack/packages/src/roboracer_gazebo/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
- link right_wheel_back: geometry collision cylinder length=0.045 radius=0.05; visual mesh filename=file:///home/dhanush/rrstack/packages/src/roboracer_gazebo/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
- link right_wheel_front: geometry collision cylinder length=0.045 radius=0.05; visual mesh filename=file:///home/dhanush/rrstack/packages/src/roboracer_gazebo/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

Commit message: Fix f110_car URDF mesh paths: replace hard-coded absolute path with portable package:// reference

File: packages/src/roboracer_gazebo/models/f110_car/f110_car.urdf (robot description, URDF)
Before this commit: robot f110_car, 12 links, 11 joints
Links:
- link camera: geometry collision box size=0.03 0.17 0.03; visual mesh filename=package://roboracer_gazebo/models/f110_car/meshes/realsense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
- link chassis: geometry collision box size=0.49 0.18 0.1; visual mesh filename=package://roboracer_gazebo/models/f110_car/meshes/car.dae
- link laser: geometry collision box size=0.1 0.1 0.1; visual mesh filename=package://roboracer_gazebo/models/f110_car/meshes/hokuyo.dae
- link left_wheel_back: geometry collision cylinder length=0.045 radius=0.05; visual mesh filename=package://roboracer_gazebo/models/f110_car/meshes/wheel.dae
- link left_wheel_front: geometry collision cylinder length=0.045 radius=0.05; visual mesh filename=package://roboracer_gazebo/models/f110_car/meshes/wheel.dae
- link right_wheel_back: geometry collision cylinder length=0.045 radius=0.05; visual mesh filename=package://roboracer_gazebo/models/f110_car/meshes/wheel.dae
- link right_wheel_front: geometry collision cylinder length=0.045 radius=0.05; visual mesh filename=package://roboracer_gazebo/models/f110_car/meshes/wheel.dae

Commit message: Assessment cycle 1: depth camera, /drive interface, world selector
URDF / simulation
- Camera switched to depth sensor (libgazebo_ros_camera, type="depth"),
  matched to RealSense D435 (640x480, ~69 deg FOV)
- RealSense-style topics: /camera/camera/color/image_raw,
  /camera/camera/depth/image_raw, /camera/camera/color/camera_info
- Added camera_color_optical_frame link + joint (image axes for tf2)
- Mesh paths changed from file:///home/... to package:// (portable)

Perception
- delaunay_node: replaced with empty stub (removes ()() crash)
- yolo_node: topic defaults match the new camera topics
- yolo_node: max_depth parameter now actually used
- yolo_node: dynamic fallback path for best.pt (next to the node file)
- Declared numpy / opencv deps, added requirements.txt (ultralytics)

Ackermann drive interface
- New package roboracer_drive_to_cmd_vel:
  /drive (AckermannDriveStamped) -> /cmd_vel (Twist), simulation only
- wall_follow_pid_node: publishes AckermannDriveStamped on /drive
- pure_pursuit_node: publishes AckermannDriveStamped on /drive
- ackermann_msgs added to package dependencies

Launch files
- gazebo.launch.py: GAZEBO_MODEL_PATH includes share dir (package:// meshes)
- gazebo.launch.py: world selector, world:=walls | cones | <path>
- wall_follow.launch.py: reuses gazebo.launch.py instead of its own Gazebo setup
- wall_follow.launch.py: starts drive_to_cmd_vel bridge with the PID node
- wall_pure_pursuit.launch.py: drive_topic argument (/drive)

Config fixes
- wall_follow_params.yaml: theta_deg -> theta_front_deg / theta_rear_deg (35 deg)
- wall_follow_params.yaml / lidar_centerline.yaml: command topic -> /drive
- roboracer_slam: added missing rviz/roboracer_slam.rviz

Known open
- wall_centerline_node still needs common.py (pure pursuit not end-to-end tested)
- Safety node, ackermann_mux, sim.launch.py: next cycle

File: packages/src/roboracer_gazebo/models/f110_car/f110_car.urdf (robot description, URDF)
Before this commit: robot f110_car, 12 links, 11 joints
Links:
- added link camera_color_optical_frame
Joints:
- added joint camera_optical_joint: type fixed, parent camera, child camera_color_optical_frame, origin xyz=0 0 0 rpy=-1.5708 0 -1.5708
